Commit message: Created core

File: description/robot_core.xacro (robot description, xacro)
@@ -15,9 +15,9 @@
    </material>
    <!-- BASE LINK-->
-   <link name= "base link">
+   <link name= "base_link">
    </link>
    <!-- CHASSIS LINK-->
-  <joint name= "chassis joint" type="fixed">
-     <parent link= "base link"/>
+  <joint name= "chassis_joint" type="fixed">
+     <parent link= "base_link"/>
      <child link="chassis"/>
      <origin xyz= "-0.1 0 0"/>
@@ -41,12 +41,15 @@
     </xacro:inertial_box>
   </link>
+  <gazebo reference="chassis">
+     <material>Gazebo/White</material>
+  </gazebo>
   <!--LEFT WHEEL LINK -->
-  <joint name="left wheel joint" type="continuous">
-      <parent link="base link"/>
-      <child link="left wheel"/>
+  <joint name="left_wheel_joint" type="continuous">
+      <parent link="base_link"/>
+      <child link="left_wheel"/>
       <origin xyz="0 0.175 0" rpy="-${pi/2} 0 0"/>
       <axis xyz="0 0 1"/>
   </joint>
-  <link name="left wheel">
+  <link name="left_wheel">
      <visual>
         <geometry>
@@ -64,12 +67,15 @@
      </xacro:inertial_cylinder>
   </link>
+  <gazebo reference="left_wheel">
+     <material>Gazebo/Blue</material>
+  </gazebo>
   <!--RIGHT WHEEL LINK -->
-  <joint name="right wheel joint" type="continuous">
-      <parent link="base link"/>
-      <child link="right wheel"/>
+  <joint name="right_wheel_joint" type="continuous">
+      <parent link="base_link"/>
+      <child link="right_wheel"/>
       <origin xyz="0 -0.175 0" rpy="${pi/2} 0 0"/>
       <axis xyz="0 0 -1"/>
   </joint>
-  <link name="right wheel">
+  <link name="right_wheel">
      <visual>
         <geometry>
@@ -87,11 +93,14 @@
      </xacro:inertial_cylinder>
   </link>
+  <gazebo reference="right_wheel">
+     <material>Gazebo/Blue</material>
+  </gazebo>
   <!-- CASTER WHEEL LINK-->
-  <joint name="caster wheel joint" type="fixed">
+  <joint name="caster_wheel_joint" type="fixed">
      <parent link="chassis"/>
-     <child link="caster wheel"/>
+     <child link="caster_wheel"/>
      <origin xyz="0.24 0 0"/>
   </joint>
-  <link name="caster wheel">
+  <link name="caster_wheel">
      <visual>
        <geometry>
@@ -109,3 +118,6 @@
      </xacro:inertial_sphere>
   </link>
+  <gazebo reference="caster_wheel">
+     <material>Gazebo/Black</material>
+  </gazebo>
 </robot>
